File: kicad/head-unit/_autosave-head-unit.kicad_sch (KiCad schematic)
At the start: 59 parts, among them J1 Debug_Port, J2 Relay_Main_Power, J3 Steering_Wheel, J4 Power Port, J5 Car Connection, J6 Relay_Ign_Detect, J7 Pi, J8 DAC+, K1 Relay_Aux_Power, K2 Relay_Amplifier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

Commit message: Initial work on headunit
Parts:
- C1: footprint Capacitor_SMD:C_0201_0603Metric -> Capacitor_SMD:C_0603_1608Metric
- C8: footprint Capacitor_SMD:C_0402_1005Metric -> Capacitor_SMD:C_1206_3216Metric
Changed lines of the file:
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@@
+    (stroke (width 0) (type default))
+  )
+  (wire (pts (xy 153.035 107.95) (xy 153.67 107.95))
     (stroke (width 0) (type default))
   )
@@
   )
   (wire (pts (xy 39.37 27.305) (xy 56.515 27.305))
+    (stroke (width 0) (type default))
+  )
+  (wire (pts (xy 153.035 107.315) (xy 153.035 107.95))
     (stroke (width 0) (type default))
   )
@@
       (effects (font (size 1.27 1.27)) (justify left))
     )
-    (property "Footprint" "Capacitor_SMD:C_0201_0603Metric" (at 120.3452 25.4 0)
+    (property "Footprint" "Capacitor_SMD:C_0603_1608Metric" (at 120.3452 25.4 0)
       (effects (font (size 1.27 1.27)) hide)
     )
@@
       (effects (font (size 1.27 1.27)) (justify left))
     )
-    (property "Footprint" "Capacitor_SMD:C_0402_1005Metric" (at 107.6452 49.53 0)
+    (property "Footprint" "Capacitor_SMD:C_1206_3216Metric" (at 107.6452 49.53 0)
       (effects (font (size 1.27 1.27)) hide)
     )
@@
     )
   )
-  (symbol (lib_id "power:GND") (at 153.67 107.95 270) (unit 1)
-    (in_bom yes) (on_board yes) (dnp no) (fields_autoplaced)
-    (property "Reference" "#PWR031" (at 147.32 107.95 0)
-      (effects (font (size 1.27 1.27)) hide)
-    )
-    (property "Value" "GND" (at 149.86 107.95 90)
-      (effects (font (size 1.27 1.27)) (justify right) hide)
-    )
-    (property "Footprint" "" (at 153.67 107.95 0)
-      (effects (font (size 1.27 1.27)) hide)
-    )
-    (property "Datasheet" "" (at 153.67 107.95 0)
-      (effects (font (size 1.27 1.27)) hide)
-    )
+  (symbol (lib_id "power:GND") (at 153.035 107.315 270) (unit 1)
+    (in_bom yes) (on_board yes) (dnp no) (fields_autoplaced)
+    (property "Reference" "#PWR031" (at 146.685 107.315 0)
+      (effects (font (size 1.27 1.27)) hide)
+    )
+    (property "Value" "GND" (at 149.225 107.315 90)
+      (effects (font (size 1.27 1.27)) (justify right) hide)
+    )
+    (property "Footprint" "" (at 153.035 107.315 0)
+      (effects (font (size 1.27 1.27)) hide)
+    )
+    (property "Datasheet" "" (at 153.035 107.315 0)
+      (effects (font (size 1.27 1.27)) hide)
+    )
