File: kicad/head-unit/12v_to_3_3v.kicad_sch (KiCad schematic)
At the start: 8 parts, among them U1 ADP1108AN-3.3

Commit message: Add I2C, begin routing
Parts:
- renumbered C8 to C16, C12 to C17, D1 to D17, L1 to L2, R1 to R22, R3 to R23, R4 to R24, U1 to U3
Changed lines of the file:
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@@
   (symbol (lib_id "power:GND") (at 106.68 71.755 0) (unit 1)
     (in_bom yes) (on_board yes) (dnp no) (fields_autoplaced)
-    (property "Reference" "#PWR010" (at 106.68 78.105 0)
+    (property "Reference" "#PWR052" (at 106.68 78.105 0)
       (effects (font (size 1.27 1.27)) hide)
     )
@@
       (project "head-unit"
         (path "/fb62c198-944e-448a-801a-748560803824/9f34b45c-ffff-4958-9323-e0ada23d6a1d"
-          (reference "#PWR010") (unit 1)
+          (reference "#PWR052") (unit 1)
         )
       )
@@
   (symbol (lib_id "Device:R") (at 157.48 104.775 0) (unit 1)
     (in_bom yes) (on_board yes) (dnp no) (fields_autoplaced)
-    (property "Reference" "R4" (at 159.385 103.505 0)
+    (property "Reference" "R24" (at 159.385 103.505 0)
       (effects (font (size 1.27 1.27)) (justify left))
     )
@@
       (project "head-unit"
         (path "/fb62c198-944e-448a-801a-748560803824/9f34b45c-ffff-4958-9323-e0ada23d6a1d"
-          (reference "R4") (unit 1)
+          (reference "R24") (unit 1)
         )
       )
@@
   (symbol (lib_id "Device:D_Schottky") (at 124.46 97.155 270) (unit 1)
     (in_bom yes) (on_board yes) (dnp no) (fields_autoplaced)
-    (property "Reference" "D1" (at 126.746 95.5675 90)
+    (property "Reference" "D17" (at 126.746 95.5675 90)
       (effects (font (size 1.27 1.27)) (justify left))
     )
@@
       (project "head-unit"
         (path "/fb62c198-944e-448a-801a-748560803824/9f34b45c-ffff-4958-9323-e0ada23d6a1d"
-          (reference "D1") (unit 1)
+          (reference "D17") (unit 1)
         )
       )
@@
   (symbol (lib_id "Device:R") (at 157.48 97.155 0) (unit 1)
     (in_bom yes) (on_board yes) (dnp no) (fields_autoplaced)
-    (property "Reference" "R3" (at 159.385 95.885 0)
+    (property "Reference" "R23" (at 159.385 95.885 0)
       (effects (font (size 1.27 1.27)) (justify left))
     )
@@
       (project "head-unit"
         (path "/fb62c198-944e-448a-801a-748560803824/9f34b45c-ffff-4958-9323-e0ada23d6a1d"
-          (reference "R3") (unit 1)
+          (reference "R23") (unit 1)
         )
       )
@@
   (symbol (lib_id "power:GND") (at 158.115 62.23 0) (unit 1)
     (in_bom yes) (on_board yes) (dnp no) (fields_autoplaced)
-    (property "Reference" "#PWR014" (at 158.115 68.58 0)
+    (property "Reference" "#PWR051" (at 158.115 68.58 0)
       (effects (font (size 1.27 1.27)) hide)
     )
@@
       (project "head-unit"
         (path "/fb62c198-944e-448a-801a-748560803824/9f34b45c-ffff-4958-9323-e0ada23d6a1d"
-          (reference "#PWR014") (unit 1)
+          (reference "#PWR051") (unit 1)
         )
       )
@@
   (symbol (lib_id "Device:R") (at 119.38 67.945 0) (unit 1)
     (in_bom yes) (on_board yes) (dnp no)
-    (property "Reference" "R1" (at 120.65 66.675 0)
+    (property "Reference" "R22" (at 120.65 66.675 0)
       (effects (font (size 1.27 1.27)) (justify left))
     )
@@
       (project "head-unit"
         (path "/fb62c198-944e-448a-801a-748560803824/9f34b45c-ffff-4958-9323-e0ada23d6a1d"
-          (reference "R1") (unit 1)
+          (reference "R22") (unit 1)
         )
       )
@@
   (symbol (lib_id "power:GND") (at 124.46 100.965 0) (unit 1)
     (in_bom yes) (on_board yes) (dnp no) (fields_autoplaced)
-    (property "Reference" "#PWR015" (at 124.46 107.315 0)
+    (property "Reference" "#PWR054" (at 124.46 107.315 0)
       (effects (font (size 1.27 1.27)) hide)
     )
@@
       (project "head-unit"
         (path "/fb62c198-944e-448a-801a-748560803824/9f34b45c-ffff-4958-9323-e0ada23d6a1d"
-          (reference "#PWR015") (unit 1)
+          (reference "#PWR054") (unit 1)
         )
       )
@@
   (symbol (lib_id "Device:C") (at 106.68 67.945 0) (unit 1)
     (in_bom yes) (on_board yes) (dnp no)
-    (property "Reference" "C8" (at 109.855 66.675 0)
+    (property "Reference" "C16" (at 109.855 66.675 0)
       (effects (font (size 1.27 1.27)) (justify left))
     )
@@
       (project "head-unit"
         (path "/fb62c198-944e-448a-801a-748560803824/9f34b45c-ffff-4958-9323-e0ada23d6a1d"
-          (reference "C8") (unit 1)
+          (reference "C16") (unit 1)
         )
       )
@@
   (symbol (lib_id "power:GND") (at 157.48 108.585 0) (unit 1)
     (in_bom yes) (on_board yes) (dnp no) (fields_autoplaced)
-    (property "Reference" "#PWR031" (at 157.48 114.935 0)
+    (property "Reference" "#PWR056" (at 157.48 114.935 0)
       (effects (font (size 1.27 1.27)) hide)
     )
@@
       (project "head-unit"
         (path "/fb62c198-944e-448a-801a-748560803824/9f34b45c-ffff-4958-9323-e0ada23d6a1d"
-          (reference "#PWR031") (unit 1)
+          (reference "#PWR056") (unit 1)
         )
       )
@@
   (symbol (lib_id "power:GND") (at 142.875 100.965 0) (unit 1)
     (in_bom yes) (on_board yes) (dnp no) (fields_autoplaced)
-    (property "Reference" "#PWR017" (at 142.875 107.315 0)
+    (property "Reference" "#PWR055" (at 142.875 107.315 0)
       (effects (font (size 1.27 1.27)) hide)
     )
@@
       (project "head-unit"
         (path "/fb62c198-944e-448a-801a-748560803824/9f34b45c-ffff-4958-9323-e0ada23d6a1d"
-          (reference "#PWR017") (unit 1)
+          (reference "#PWR055") (unit 1)
         )
       )
@@
   (symbol (lib_id "Device:L") (at 139.065 93.345 90) (unit 1)
     (in_bom yes) (on_board yes) (dnp no)
-    (property "Reference" "L1" (at 139.319 91.313 90)
+    (property "Reference" "L2" (at 139.319 91.313 90)
       (effects (font (size 1.27 1.27)))
     )
@@
       (project "head-unit"
         (path "/fb62c198-944e-448a-801a-748560803824/9f34b45c-ffff-4958-9323-e0ada23d6a1d"
-          (reference "L1") (unit 1)
+          (reference "L2") (unit 1)
         )
       )
@@
   (symbol (lib_id "Regulator_Switching:ADP1108AN-3.3") (at 124.46 83.185 0) (unit 1)
     (in_bom yes) (on_board yes) (dnp no)
-    (property "Reference" "U1" (at 111.76 79.375 0)
+    (property "Reference" "U3" (at 111.76 79.375 0)
       (effects (font (size 1.27 1.27)))
     )
@@
       (project "head-unit"
         (path "/fb62c198-944e-448a-801a-748560803824/9f34b45c-ffff-4958-9323-e0ada23d6a1d"
-          (reference "U1") (unit 1)
+          (reference "U3") (unit 1)
         )
       )
@@
   (symbol (lib_id "Device:C") (at 142.875 97.155 0) (unit 1)
     (in_bom yes) (on_board yes) (dnp no)
-    (property "Reference" "C12" (at 146.685 95.885 0)
+    (property "Reference" "C17" (at 146.685 95.885 0)
       (effects (font (size 1.27 1.27)) (justify left))
     )
@@
       (project "head-unit"
         (path "/fb62c198-944e-448a-801a-748560803824/9f34b45c-ffff-4958-9323-e0ada23d6a1d"
-          (reference "C12") (unit 1)
+          (reference "C17") (unit 1)
         )
       )
@@
   (symbol (lib_id "power:GND") (at 119.38 93.345 0) (unit 1)
     (in_bom yes) (on_board yes) (dnp no) (fields_autoplaced)
-    (property "Reference" "#PWR011" (at 119.38 99.695 0)
+    (property "Reference" "#PWR053" (at 119.38 99.695 0)
       (effects (font (size 1.27 1.27)) hide)
     )
@@
       (project "head-unit"
         (path "/fb62c198-944e-448a-801a-748560803824/9f34b45c-ffff-4958-9323-e0ada23d6a1d"
-          (reference "#PWR011") (unit 1)
-        )
-      )
+          (reference "#PWR053") (unit 1)
+        )
+      )

Commit message: WIP routing
Parts:
- R23, R24: footprint Resistor_SMD:R_0402_1005Metric -> Resistor_SMD:R_0603_1608Metric
Changed lines of the file:
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@@
       (effects (font (size 1.27 1.27)) (justify left))
     )
-    (property "Footprint" "Resistor_SMD:R_0402_1005Metric" (at 155.702 104.775 90)
+    (property "Footprint" "Resistor_SMD:R_0603_1608Metric" (at 155.702 104.775 90)
       (effects (font (size 1.27 1.27)) hide)
     )
@@
       (effects (font (size 1.27 1.27)) (justify left))
     )
-    (property "Footprint" "Resistor_SMD:R_0402_1005Metric" (at 155.702 97.155 90)
+    (property "Footprint" "Resistor_SMD:R_0603_1608Metric" (at 155.702 97.155 90)
       (effects (font (size 1.27 1.27)) hide)
     )
