File: kicad/head-unit/12v_to_5v.kicad_sch (KiCad schematic)
At the start: 11 parts, among them U3 TPS56339DDC

Commit message: Fix mosfets, switch to screw terminals and XT60
Parts:
- C10, C13, C15, C16: footprint (none) -> Capacitor_SMD:C_0603_1608Metric
- C14, C17: footprint (none) -> Capacitor_SMD:C_0402_1005Metric
- L2: footprint (none) -> Inductor_SMD:L_6.3x6.3_H3
- R5: footprint (none) -> Resistor_SMD:R_0402_1005Metric
- R6: footprint (none) -> Resistor_SMD:R_0612_1632Metric
- R7: footprint (none) -> Resistor_SMD:R_0201_0603Metric

Commit message: Add I2C, begin routing
Parts:
- renumbered C14 to C10, C10 to C11, C16 to C12, C17 to C13, C13 to C14, L2 to L1, R7 to R19, R6 to R20, R5 to R21, U3 to U2
Changed lines of the file:
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@@
   (symbol (lib_id "Device:L") (at 163.195 72.39 90) (unit 1)
     (in_bom yes) (on_board yes) (dnp no)
-    (property "Reference" "L2" (at 163.195 70.485 90)
+    (property "Reference" "L1" (at 163.195 70.485 90)
       (effects (font (size 1.27 1.27)))
     )
@@
       (project "head-unit"
         (path "/fb62c198-944e-448a-801a-748560803824/7e6b7ef7-bd1e-41c9-940e-1581ef719381"
-          (reference "L2") (unit 1)
+          (reference "L1") (unit 1)
         )
       )
@@
   (symbol (lib_id "power:GND") (at 187.96 80.645 0) (unit 1)
     (in_bom yes) (on_board yes) (dnp no) (fields_autoplaced)
-    (property "Reference" "#PWR032" (at 187.96 86.995 0)
+    (property "Reference" "#PWR048" (at 187.96 86.995 0)
       (effects (font (size 1.27 1.27)) hide)
     )
@@
       (project "head-unit"
         (path "/fb62c198-944e-448a-801a-748560803824/7e6b7ef7-bd1e-41c9-940e-1581ef719381"
-          (reference "#PWR032") (unit 1)
+          (reference "#PWR048") (unit 1)
         )
       )
@@
   (symbol (lib_id "Device:C") (at 97.155 73.66 0) (unit 1)
     (in_bom yes) (on_board yes) (dnp no)
-    (property "Reference" "C10" (at 97.79 71.755 0)
+    (property "Reference" "C11" (at 97.79 71.755 0)
       (effects (font (size 1.27 1.27)) (justify left))
     )
@@
       (project "head-unit"
         (path "/fb62c198-944e-448a-801a-748560803824/7e6b7ef7-bd1e-41c9-940e-1581ef719381"
-          (reference "C10") (unit 1)
+          (reference "C11") (unit 1)
         )
       )
@@
   (symbol (lib_id "Device:C") (at 178.435 76.2 0) (unit 1)
     (in_bom yes) (on_board yes) (dnp no) (fields_autoplaced)
-    (property "Reference" "C13" (at 181.61 74.93 0)
+    (property "Reference" "C14" (at 181.61 74.93 0)
       (effects (font (size 1.27 1.27)) (justify left))
     )
@@
       (project "head-unit"
         (path "/fb62c198-944e-448a-801a-748560803824/7e6b7ef7-bd1e-41c9-940e-1581ef719381"
-          (reference "C13") (unit 1)
+          (reference "C14") (unit 1)
         )
       )
@@
   (symbol (lib_id "power:GND") (at 178.435 80.645 0) (unit 1)
     (in_bom yes) (on_board yes) (dnp no) (fields_autoplaced)
-    (property "Reference" "#PWR030" (at 178.435 86.995 0)
+    (property "Reference" "#PWR047" (at 178.435 86.995 0)
       (effects (font (size 1.27 1.27)) hide)
     )
@@
       (project "head-unit"
         (path "/fb62c198-944e-448a-801a-748560803824/7e6b7ef7-bd1e-41c9-940e-1581ef719381"
-          (reference "#PWR030") (unit 1)
+          (reference "#PWR047") (unit 1)
         )
       )
@@
   (symbol (lib_id "Device:R") (at 145.415 72.39 90) (unit 1)
     (in_bom yes) (on_board yes) (dnp no) (fields_autoplaced)
-    (property "Reference" "R7" (at 145.415 66.04 90)
+    (property "Reference" "R19" (at 145.415 66.04 90)
       (effects (font (size 1.27 1.27)))
     )
@@
       (project "head-unit"
         (path "/fb62c198-944e-448a-801a-748560803824/7e6b7ef7-bd1e-41c9-940e-1581ef719381"
-          (reference "R7") (unit 1)
+          (reference "R19") (unit 1)
         )
       )
@@
   (symbol (lib_id "Device:C") (at 110.49 73.66 0) (unit 1)
     (in_bom yes) (on_board yes) (dnp no)
-    (property "Reference" "C17" (at 111.76 71.755 0)
+    (property "Reference" "C13" (at 111.76 71.755 0)
       (effects (font (size 1.27 1.27)) (justify left))
     )
@@
       (project "head-unit"
         (path "/fb62c198-944e-448a-801a-748560803824/7e6b7ef7-bd1e-41c9-940e-1581ef719381"
-          (reference "C17") (unit 1)
+          (reference "C13") (unit 1)
         )
       )
@@
   (symbol (lib_id "Device:R") (at 167.005 83.82 0) (unit 1)
     (in_bom yes) (on_board yes) (dnp no) (fields_autoplaced)
-    (property "Reference" "R5" (at 168.91 82.55 0)
+    (property "Reference" "R21" (at 168.91 82.55 0)
       (effects (font (size 1.27 1.27)) (justify left))
     )
@@
       (project "head-unit"
         (path "/fb62c198-944e-448a-801a-748560803824/7e6b7ef7-bd1e-41c9-940e-1581ef719381"
-          (reference "R5") (unit 1)
+          (reference "R21") (unit 1)
         )
       )
@@
   (symbol (lib_id "Device:C") (at 103.505 73.66 0) (unit 1)
     (in_bom yes) (on_board yes) (dnp no)
-    (property "Reference" "C16" (at 104.14 71.755 0)
+    (property "Reference" "C12" (at 104.14 71.755 0)
       (effects (font (size 1.27 1.27)) (justify left))
     )
@@
       (project "head-unit"
         (path "/fb62c198-944e-448a-801a-748560803824/7e6b7ef7-bd1e-41c9-940e-1581ef719381"
-          (reference "C16") (unit 1)
+          (reference "C12") (unit 1)
         )
       )
@@
   (symbol (lib_id "Device:R") (at 167.005 76.2 0) (unit 1)
     (in_bom yes) (on_board yes) (dnp no) (fields_autoplaced)
-    (property "Reference" "R6" (at 168.91 74.93 0)
+    (property "Reference" "R20" (at 168.91 74.93 0)
       (effects (font (size 1.27 1.27)) (justify left))
     )
@@
       (project "head-unit"
         (path "/fb62c198-944e-448a-801a-748560803824/7e6b7ef7-bd1e-41c9-940e-1581ef719381"
-          (reference "R6") (unit 1)
+          (reference "R20") (unit 1)
         )
       )
@@
   (symbol (lib_id "power:GND") (at 167.005 88.265 0) (unit 1)
     (in_bom yes) (on_board yes) (dnp no) (fields_autoplaced)
-    (property "Reference" "#PWR029" (at 167.005 94.615 0)
+    (property "Reference" "#PWR050" (at 167.005 94.615 0)
       (effects (font (size 1.27 1.27)) hide)
     )
@@
       (project "head-unit"
         (path "/fb62c198-944e-448a-801a-748560803824/7e6b7ef7-bd1e-41c9-940e-1581ef719381"
-          (reference "#PWR029") (unit 1)
+          (reference "#PWR050") (unit 1)
         )
       )
@@
   (symbol (lib_id "power:GND") (at 110.49 80.645 0) (unit 1)
     (in_bom yes) (on_board yes) (dnp no) (fields_autoplaced)
-    (property "Reference" "#PWR028" (at 110.49 86.995 0)
+    (property "Reference" "#PWR046" (at 110.49 86.995 0)
       (effects (font (size 1.27 1.27)) hide)
     )
@@
       (project "head-unit"
         (path "/fb62c198-944e-448a-801a-748560803824/7e6b7ef7-bd1e-41c9-940e-1581ef719381"
-          (reference "#PWR028") (unit 1)
+          (reference "#PWR046") (unit 1)
         )
       )
@@
   (symbol (lib_id "Device:C") (at 155.575 72.39 90) (unit 1)
     (in_bom yes) (on_board yes) (dnp no) (fields_autoplaced)
-    (property "Reference" "C14" (at 155.575 64.77 90)
+    (property "Reference" "C10" (at 155.575 64.77 90)
       (effects (font (size 1.27 1.27)))
     )
@@
       (project "head-unit"
         (path "/fb62c198-944e-448a-801a-748560803824/7e6b7ef7-bd1e-41c9-940e-1581ef719381"
-          (reference "C14") (unit 1)
+          (reference "C10") (unit 1)
         )
       )
@@
   (symbol (lib_id "power:GND") (at 129.54 81.915 0) (unit 1)
     (in_bom yes) (on_board yes) (dnp no) (fields_autoplaced)
-    (property "Reference" "#PWR027" (at 129.54 88.265 0)
+    (property "Reference" "#PWR049" (at 129.54 88.265 0)
       (effects (font (size 1.27 1.27)) hide)
     )
@@
       (project "head-unit"
         (path "/fb62c198-944e-448a-801a-748560803824/7e6b7ef7-bd1e-41c9-940e-1581ef719381"
-          (reference "#PWR027") (unit 1)
+          (reference "#PWR049") (unit 1)
         )
       )
@@
   (symbol (lib_id "power:GND") (at 97.79 57.15 0) (unit 1)
     (in_bom yes) (on_board yes) (dnp no) (fields_autoplaced)
-    (property "Reference" "#PWR068" (at 97.79 63.5 0)
+    (property "Reference" "#PWR045" (at 97.79 63.5 0)
       (effects (font (size 1.27 1.27)) hide)
     )
@@
       (project "head-unit"
         (path "/fb62c198-944e-448a-801a-748560803824/7e6b7ef7-bd1e-41c9-940e-1581ef719381"
-          (reference "#PWR068") (unit 1)
+          (reference "#PWR045") (unit 1)
         )
       )
@@
   (symbol (lib_id "Regulator_Switching:TPS56339DDC") (at 129.54 72.39 0) (unit 1)
     (in_bom yes) (on_board yes) (dnp no) (fields_autoplaced)
-    (property "Reference" "U3" (at 129.54 62.23 0)
+    (property "Reference" "U2" (at 129.54 62.23 0)
       (effects (font (size 1.27 1.27)))
     )
@@
       (project "head-unit"
         (path "/fb62c198-944e-448a-801a-748560803824/7e6b7ef7-bd1e-41c9-940e-1581ef719381"
-          (reference "U3") (unit 1)
-        )
-      )
+          (reference "U2") (unit 1)
+        )
+      )

Commit message: WIP routing
Parts:
- R20: footprint Resistor_SMD:R_0612_1632Metric -> Resistor_SMD:R_0805_2012Metric
- R21: footprint Resistor_SMD:R_0402_1005Metric -> Resistor_SMD:R_0603_1608Metric
Changed lines of the file:
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@@
       (effects (font (size 1.27 1.27)) (justify left))
     )
-    (property "Footprint" "Resistor_SMD:R_0402_1005Metric" (at 165.227 83.82 90)
+    (property "Footprint" "Resistor_SMD:R_0603_1608Metric" (at 165.227 83.82 90)
       (effects (font (size 1.27 1.27)) hide)
     )
@@
       (effects (font (size 1.27 1.27)) (justify left))
     )
-    (property "Footprint" "Resistor_SMD:R_0612_1632Metric" (at 165.227 76.2 90)
+    (property "Footprint" "Resistor_SMD:R_0805_2012Metric" (at 165.227 76.2 90)
       (effects (font (size 1.27 1.27)) hide)
     )
